File: Hardware/analog-clock-module/analog-clock-module.kicad_pcb (KiCad board)
At the start: 2 copper layers, 300 x 300 mm, 100 parts

Commit message: bump
Connections:
- D1010 pad 1: unconnected-(D1010-DOUT-Pad1) -> /Hour2/Clock Inner Hand2/DOUT
- D1110 pad 1: unconnected-(D1110-DOUT-Pad1) -> /Hour2/DOUT
- D1210 pad 1: unconnected-(D1210-DOUT-Pad1) -> /Hour2/Clock Inner Hand3/DOUT
- D1310 pad 1: unconnected-(D1310-DOUT-Pad1) -> /Hour2/Clock Inner Hand4/DOUT
- D210 pad 1: unconnected-(D210-DOUT-Pad1) -> /Hour1/Clock Inner Hand1/DOUT
- D310 pad 1: unconnected-(D310-DOUT-Pad1) -> /Hour1/Clock Inner Hand2/DOUT
- D510 pad 1: unconnected-(D510-DOUT-Pad1) -> /Hour1/Clock Inner Hand3/DOUT
- D610 pad 1: unconnected-(D610-DOUT-Pad1) -> /Hour1/Clock Inner Hand4/DOUT
- D710 pad 1: unconnected-(D710-DOUT-Pad1) -> /Hour1/DOUT
- D910 pad 1: unconnected-(D910-DOUT-Pad1) -> /Hour2/Clock Inner Hand1/DOUT
Routing:
- net /Hour1/Clock Inner Hand4/DOUT: track 0.00 -> 176.7 mm
- net /Hour1/Clock Inner Hand2/DOUT: track 0.00 -> 88.5 mm
- net /Hour1/Clock Inner Hand3/DOUT: track 0.00 -> 88.4 mm
- net /Hour1/Clock Inner Hand1/DOUT: track 0.00 -> 88.4 mm
- net /Hour2/DOUT: track 0.00 -> 88.4 mm
- net /Hour2/Clock Inner Hand2/DOUT: track 0.00 -> 88.4 mm
- net /Hour2/Clock Inner Hand3/DOUT: track 0.00 -> 88.4 mm
- net /Hour2/Clock Inner Hand4/DOUT: track 0.00 -> 88.4 mm
- net /Hour2/Clock Inner Hand1/DOUT: track 0.00 -> 88.2 mm

Commit message: full quadrant
Parts:
- added D1601: NeoPixel_THT, LED_THT:LED_D5.0mm-4_RGB, F.Cu at (57.7, -27.6)
- added D1602: NeoPixel_THT, LED_THT:LED_D5.0mm-4_RGB, F.Cu at (65.0, -30.9)
- added D1603: NeoPixel_THT, LED_THT:LED_D5.0mm-4_RGB, F.Cu at (72.3, -34.1)
- added D1604: NeoPixel_THT, LED_THT:LED_D5.0mm-4_RGB, F.Cu at (79.6, -37.4)
- added D1605: NeoPixel_THT, LED_THT:LED_D5.0mm-4_RGB, F.Cu at (86.9, -40.6)
- added D1606: NeoPixel_THT, LED_THT:LED_D5.0mm-4_RGB, F.Cu at (94.2, -43.9)
- added D1607: NeoPixel_THT, LED_THT:LED_D5.0mm-4_RGB, F.Cu at (101.5, -47.1)
- added D1608: NeoPixel_THT, LED_THT:LED_D5.0mm-4_RGB, F.Cu at (108.8, -50.4)
- added D1609: NeoPixel_THT, LED_THT:LED_D5.0mm-4_RGB, F.Cu at (116.1, -53.6)
- added D1610: NeoPixel_THT, LED_THT:LED_D5.0mm-4_RGB, F.Cu at (123.5, -56.9)
- added D1701: NeoPixel_THT, LED_THT:LED_D5.0mm-4_RGB, F.Cu at (54.5, -33.6)
- added D1702: NeoPixel_THT, LED_THT:LED_D5.0mm-4_RGB, F.Cu at (61.4, -37.6)
- added D1703: NeoPixel_THT, LED_THT:LED_D5.0mm-4_RGB, F.Cu at (68.3, -41.6)
- added D1704: NeoPixel_THT, LED_THT:LED_D5.0mm-4_RGB, F.Cu at (75.3, -45.6)
- added D1705: NeoPixel_THT, LED_THT:LED_D5.0mm-4_RGB, F.Cu at (82.2, -49.6)
- added D1706: NeoPixel_THT, LED_THT:LED_D5.0mm-4_RGB, F.Cu at (89.1, -53.6)
- added D1707: NeoPixel_THT, LED_THT:LED_D5.0mm-4_RGB, F.Cu at (96.0, -57.6)
- added D1708: NeoPixel_THT, LED_THT:LED_D5.0mm-4_RGB, F.Cu at (103.0, -61.6)
- added D1709: NeoPixel_THT, LED_THT:LED_D5.0mm-4_RGB, F.Cu at (109.9, -65.6)
- added D1710: NeoPixel_THT, LED_THT:LED_D5.0mm-4_RGB, F.Cu at (116.8, -69.6)
- added D1801: NeoPixel_THT, LED_THT:LED_D5.0mm-4_RGB, F.Cu at (62.2, -15.1)
- added D1802: NeoPixel_THT, LED_THT:LED_D5.0mm-4_RGB, F.Cu at (70.0, -16.7)
- added D1803: NeoPixel_THT, LED_THT:LED_D5.0mm-4_RGB, F.Cu at (77.8, -18.4)
- added D1804: NeoPixel_THT, LED_THT:LED_D5.0mm-4_RGB, F.Cu at (85.6, -20.0)
- added D1805: NeoPixel_THT, LED_THT:LED_D5.0mm-4_RGB, F.Cu at (93.5, -21.7)
- added D1806: NeoPixel_THT, LED_THT:LED_D5.0mm-4_RGB, F.Cu at (101.3, -23.4)
- added D1807: NeoPixel_THT, LED_THT:LED_D5.0mm-4_RGB, F.Cu at (109.1, -25.0)
- added D1808: NeoPixel_THT, LED_THT:LED_D5.0mm-4_RGB, F.Cu at (116.9, -26.7)
- added D1809: NeoPixel_THT, LED_THT:LED_D5.0mm-4_RGB, F.Cu at (124.8, -28.4)
- added D1810: NeoPixel_THT, LED_THT:LED_D5.0mm-4_RGB, F.Cu at (132.6, -30.0)
- added D1901: NeoPixel_THT, LED_THT:LED_D5.0mm-4_RGB, F.Cu at (63.4, -8.47)
- added D1902: NeoPixel_THT, LED_THT:LED_D5.0mm-4_RGB, F.Cu at (71.3, -9.31)
- added D1903: NeoPixel_THT, LED_THT:LED_D5.0mm-4_RGB, F.Cu at (79.3, -10.1)
- added D1904: NeoPixel_THT, LED_THT:LED_D5.0mm-4_RGB, F.Cu at (87.2, -11.0)
- added D1905: NeoPixel_THT, LED_THT:LED_D5.0mm-4_RGB, F.Cu at (95.2, -11.8)
- added D1906: NeoPixel_THT, LED_THT:LED_D5.0mm-4_RGB, F.Cu at (103.1, -12.7)
- added D1907: NeoPixel_THT, LED_THT:LED_D5.0mm-4_RGB, F.Cu at (111.1, -13.5)
- added D1908: NeoPixel_THT, LED_THT:LED_D5.0mm-4_RGB, F.Cu at (119.1, -14.3)
- added D1909: NeoPixel_THT, LED_THT:LED_D5.0mm-4_RGB, F.Cu at (127.0, -15.2)
- added D1910: NeoPixel_THT, LED_THT:LED_D5.0mm-4_RGB, F.Cu at (135.0, -16.0)
- added D2001: NeoPixel_THT, LED_THT:LED_D5.0mm-4_RGB, F.Cu at (60.2, -21.5)
- added D2002: NeoPixel_THT, LED_THT:LED_D5.0mm-4_RGB, F.Cu at (67.9, -24.0)
- added D2003: NeoPixel_THT, LED_THT:LED_D5.0mm-4_RGB, F.Cu at (75.5, -26.4)
- added D2004: NeoPixel_THT, LED_THT:LED_D5.0mm-4_RGB, F.Cu at (83.1, -28.9)
- added D2005: NeoPixel_THT, LED_THT:LED_D5.0mm-4_RGB, F.Cu at (90.7, -31.4)
- added D2006: NeoPixel_THT, LED_THT:LED_D5.0mm-4_RGB, F.Cu at (98.3, -33.8)
- added D2007: NeoPixel_THT, LED_THT:LED_D5.0mm-4_RGB, F.Cu at (105.9, -36.3)
- added D2008: NeoPixel_THT, LED_THT:LED_D5.0mm-4_RGB, F.Cu at (113.5, -38.8)
- added D2009: NeoPixel_THT, LED_THT:LED_D5.0mm-4_RGB, F.Cu at (121.1, -41.3)
- added D2010: NeoPixel_THT, LED_THT:LED_D5.0mm-4_RGB, F.Cu at (128.7, -43.7)
Connections:
- net /Hour1/Clock Inner Hand1/DOUT renamed /Quadrant/Hour1/Clock Inner Hand1/DOUT
- net /Hour1/Clock Inner Hand2/DOUT renamed /Quadrant/Hour1/Clock Inner Hand2/DOUT
- net /Hour1/Clock Inner Hand3/DOUT renamed /Quadrant/Hour1/Clock Inner Hand3/DOUT
- net /Hour1/Clock Inner Hand4/DOUT renamed /Quadrant/Hour1/Clock Inner Hand4/DOUT
- net /Hour1/DIN renamed /Quadrant/Hour1/DIN
- net /Hour2/Clock Inner Hand1/DOUT renamed /Quadrant/Hour2/Clock Inner Hand1/DOUT
- net /Hour2/Clock Inner Hand2/DOUT renamed /Quadrant/Hour2/Clock Inner Hand2/DOUT
- net /Hour2/Clock Inner Hand3/DOUT renamed /Quadrant/Hour2/Clock Inner Hand3/DOUT
- net /Hour2/Clock Inner Hand4/DOUT renamed /Quadrant/Hour2/Clock Inner Hand4/DOUT
- D1110 pad 1: /Hour2/DOUT -> /Quadrant/Hour2/DOUT
- D710 pad 1: /Hour1/DOUT -> /Quadrant/Hour1/DOUT
- D901 pad 4: /Hour2/DIN -> /Quadrant/Hour1/DOUT
Routing:
- net +5V: track 719.0 -> 1078.5 mm
- net /Quadrant/Hour3/Clock Inner Hand2/DOUT: track 0.00 -> 88.5 mm
- net /Quadrant/Hour3/Clock Inner Hand3/DOUT: track 0.00 -> 88.4 mm
- net /Quadrant/Hour3/Clock Inner Hand1/DOUT: track 0.00 -> 88.4 mm
- net /Quadrant/Hour2/DOUT: track 0.00 -> 88.4 mm
- net /Hour2/DOUT: track 88.4 -> 0.00 mm
- net /Quadrant/Hour1/Clock Inner Hand4/DOUT: track 176.7 -> 88.3 mm
- net /Quadrant/Hour1/DOUT: track 0.00 -> 88.4 mm
- net /Quadrant/Hour3/Clock Inner Hand4/DOUT: track 0.00 -> 88.3 mm
- net /Quadrant/Hour3/DOUT: track 0.00 -> 81.5 mm
- net Net-(D1801-DOUT): track 0.00 -> 9.62 mm
- net Net-(D2009-DOUT): track 0.00 -> 9.62 mm
- net Net-(D1601-DOUT): track 0.00 -> 9.62 mm
- net Net-(D1809-DOUT): track 0.00 -> 9.62 mm
- net Net-(D1609-DOUT): track 0.00 -> 9.62 mm
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Other:
- board outline removed
