File: Hardware/analog-clock-module/analog-clock-module.kicad_sch (KiCad schematic)
At the start: 0 parts

Commit message: add all components and inital project layout
Other:
- added sheet Hour1 (hour.kicad_sch)
- added sheet Hour2 (hour.kicad_sch)
Changed lines of the file:
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@@
     (company "ac1ja")
+  )
+  (sheet (at 132.08 27.94) (size 19.05 7.62) (fields_autoplaced)
+    (stroke (width 0.1524) (type solid))
+    (fill (color 0 0 0 0.0000))
+    (property "Sheetname" "Hour1" (at 132.08 27.2284 0)
+      (effects (font (size 1.27 1.27)) (justify left bottom))
+    )
+    (property "Sheetfile" "hour.kicad_sch" (at 132.08 36.1446 0)
+      (effects (font (size 1.27 1.27)) (justify left top))
+    )
+    (pin "DIN" input (at 132.08 31.75 180)
+      (effects (font (size 1.27 1.27)) (justify left))
+    )
+    (pin "DOUT" output (at 151.13 31.75 0)
+      (effects (font (size 1.27 1.27)) (justify right))
+    )
+    (instances
+      (project "analog-clock-module"
+        (path "/894f620e-3404-4a40-a2a7-513bc1d5f99b" (page "4"))
+      )
+    )
+  )
+  (sheet (at 132.08 40.64) (size 19.05 7.62) (fields_autoplaced)
+    (stroke (width 0.1524) (type solid))
+    (fill (color 0 0 0 0.0000))
+    (property "Sheetname" "Hour2" (at 132.08 39.9284 0)
+      (effects (font (size 1.27 1.27)) (justify left bottom))
+    )
+    (property "Sheetfile" "hour.kicad_sch" (at 132.08 48.8446 0)
+      (effects (font (size 1.27 1.27)) (justify left top))
+    )
+    (pin "DIN" input (at 132.08 44.45 180)
+      (effects (font (size 1.27 1.27)) (justify left))
+    )
+    (pin "DOUT" output (at 151.13 44.45 0)
+      (effects (font (size 1.27 1.27)) (justify right))
+    )
+    (instances
+      (project "analog-clock-module"
+        (path "/894f620e-3404-4a40-a2a7-513bc1d5f99b" (page "8"))
+      )
+    )
   )
   (sheet_instances

Commit message: bump
Changed lines of the file:
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@@
     (company "ac1ja")
+  )
+  (wire (pts (xy 129.54 39.37) (xy 129.54 46.99))
+    (stroke (width 0) (type default))
+  )
+  (wire (pts (xy 153.67 31.75) (xy 153.67 39.37))
+    (stroke (width 0) (type default))
+  )
+  (wire (pts (xy 129.54 46.99) (xy 132.08 46.99))
+    (stroke (width 0) (type default))
+  )
+  (wire (pts (xy 151.13 31.75) (xy 153.67 31.75))
+    (stroke (width 0) (type default))
+  )
+  (wire (pts (xy 153.67 39.37) (xy 129.54 39.37))
+    (stroke (width 0) (type default))
   )
   (sheet (at 132.08 27.94) (size 19.05 7.62) (fields_autoplaced)
@@
     )
   )
-  (sheet (at 132.08 40.64) (size 19.05 7.62) (fields_autoplaced)
+  (sheet (at 132.08 43.18) (size 19.05 7.62) (fields_autoplaced)
     (stroke (width 0.1524) (type solid))
     (fill (color 0 0 0 0.0000))
-    (property "Sheetname" "Hour2" (at 132.08 39.9284 0)
+    (property "Sheetname" "Hour2" (at 132.08 42.4684 0)
       (effects (font (size 1.27 1.27)) (justify left bottom))
     )
-    (property "Sheetfile" "hour.kicad_sch" (at 132.08 48.8446 0)
+    (property "Sheetfile" "hour.kicad_sch" (at 132.08 51.3846 0)
       (effects (font (size 1.27 1.27)) (justify left top))
     )
-    (pin "DIN" input (at 132.08 44.45 180)
+    (pin "DIN" input (at 132.08 46.99 180)
       (effects (font (size 1.27 1.27)) (justify left))
     )
-    (pin "DOUT" output (at 151.13 44.45 0)
+    (pin "DOUT" output (at 151.13 46.99 0)
       (effects (font (size 1.27 1.27)) (justify right))
     )

Commit message: full quadrant
Other:
- removed sheet Hour1
- removed sheet Hour2
- added sheet Quadrant (quadrant.kicad_sch)
Changed lines of the file:
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@@
     (company "ac1ja")
   )
-  (wire (pts (xy 129.54 39.37) (xy 129.54 46.99))
-    (stroke (width 0) (type default))
-  )
-  (wire (pts (xy 153.67 31.75) (xy 153.67 39.37))
-    (stroke (width 0) (type default))
-  )
-  (wire (pts (xy 129.54 46.99) (xy 132.08 46.99))
-    (stroke (width 0) (type default))
-  )
-  (wire (pts (xy 151.13 31.75) (xy 153.67 31.75))
-    (stroke (width 0) (type default))
-  )
-  (wire (pts (xy 153.67 39.37) (xy 129.54 39.37))
-    (stroke (width 0) (type default))
-  )
-  (sheet (at 132.08 27.94) (size 19.05 7.62) (fields_autoplaced)
+  (sheet (at 144.78 34.29) (size 21.59 10.16) (fields_autoplaced)
     (stroke (width 0.1524) (type solid))
     (fill (color 0 0 0 0.0000))
-    (property "Sheetname" "Hour1" (at 132.08 27.2284 0)
+    (property "Sheetname" "Quadrant" (at 144.78 33.5784 0)
       (effects (font (size 1.27 1.27)) (justify left bottom))
     )
-    (property "Sheetfile" "hour.kicad_sch" (at 132.08 36.1446 0)
+    (property "Sheetfile" "quadrant.kicad_sch" (at 144.78 45.0346 0)
       (effects (font (size 1.27 1.27)) (justify left top))
     )
-    (pin "DIN" input (at 132.08 31.75 180)
+    (pin "DIN" input (at 144.78 39.37 180)
       (effects (font (size 1.27 1.27)) (justify left))
     )
-    (pin "DOUT" output (at 151.13 31.75 0)
+    (pin "DOUT" output (at 166.37 39.37 0)
       (effects (font (size 1.27 1.27)) (justify right))
     )
     (instances
       (project "analog-clock-module"
-        (path "/894f620e-3404-4a40-a2a7-513bc1d5f99b" (page "4"))
+        (path "/894f620e-3404-4a40-a2a7-513bc1d5f99b" (page "2"))
       )
     )
-  )
-  (sheet (at 132.08 43.18) (size 19.05 7.62) (fields_autoplaced)
-    (stroke (width 0.1524) (type solid))
-    (fill (color 0 0 0 0.0000))
-    (property "Sheetname" "Hour2" (at 132.08 42.4684 0)
-      (effects (font (size 1.27 1.27)) (justify left bottom))
-    )
-    (property "Sheetfile" "hour.kicad_sch" (at 132.08 51.3846 0)
-      (effects (font (size 1.27 1.27)) (justify left top))
-    )
-    (pin "DIN" input (at 132.08 46.99 180)
-      (effects (font (size 1.27 1.27)) (justify left))
-    )
-    (pin "DOUT" output (at 151.13 46.99 0)
-      (effects (font (size 1.27 1.27)) (justify right))
-    )
-    (instances
-      (project "analog-clock-module"
-        (path "/894f620e-3404-4a40-a2a7-513bc1d5f99b" (page "8"))
-      )
-    )

Commit message: All done
Other:
- sheet Quadrant renamed Quadrant1
- added sheet Quadrant2 (quadrant.kicad_sch)
- added sheet Quadrant3 (quadrant.kicad_sch)
- added sheet Quadrant4 (quadrant.kicad_sch)
Changed lines of the file:
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@@
     (company "ac1ja")
+  )
+  (wire (pts (xy 166.37 77.47) (xy 170.18 77.47))
+    (stroke (width 0) (type default))
+  )
+  (wire (pts (xy 166.37 58.42) (xy 170.18 58.42))
+    (stroke (width 0) (type default))
+  )
+  (wire (pts (xy 140.97 58.42) (xy 144.78 58.42))
+    (stroke (width 0) (type default))
+  )
+  (wire (pts (xy 140.97 96.52) (xy 144.78 96.52))
+    (stroke (width 0) (type default))
+  )
+  (wire (pts (xy 140.97 87.63) (xy 140.97 96.52))
+    (stroke (width 0) (type default))
+  )
+  (wire (pts (xy 140.97 77.47) (xy 144.78 77.47))
+    (stroke (width 0) (type default))
+  )
+  (wire (pts (xy 166.37 39.37) (xy 170.18 39.37))
+    (stroke (width 0) (type default))
+  )
+  (wire (pts (xy 140.97 49.53) (xy 140.97 58.42))
+    (stroke (width 0) (type default))
+  )
+  (wire (pts (xy 170.18 49.53) (xy 140.97 49.53))
+    (stroke (width 0) (type default))
+  )
+  (wire (pts (xy 170.18 39.37) (xy 170.18 49.53))
+    (stroke (width 0) (type default))
+  )
+  (wire (pts (xy 170.18 68.58) (xy 140.97 68.58))
+    (stroke (width 0) (type default))
+  )
+  (wire (pts (xy 170.18 58.42) (xy 170.18 68.58))
+    (stroke (width 0) (type default))
+  )
+  (wire (pts (xy 140.97 68.58) (xy 140.97 77.47))
+    (stroke (width 0) (type default))
+  )
+  (wire (pts (xy 170.18 77.47) (xy 170.18 87.63))
+    (stroke (width 0) (type default))
+  )
+  (wire (pts (xy 170.18 87.63) (xy 140.97 87.63))
+    (stroke (width 0) (type default))
   )
   (sheet (at 144.78 34.29) (size 21.59 10.16) (fields_autoplaced)
     (stroke (width 0.1524) (type solid))
     (fill (color 0 0 0 0.0000))
-    (property "Sheetname" "Quadrant" (at 144.78 33.5784 0)
+    (property "Sheetname" "Quadrant1" (at 144.78 33.5784 0)
       (effects (font (size 1.27 1.27)) (justify left bottom))
     )
@@
       )
     )
+  )
+  (sheet (at 144.78 72.39) (size 21.59 10.16) (fields_autoplaced)
+    (stroke (width 0.1524) (type solid))
+    (fill (color 0 0 0 0.0000))
+    (property "Sheetname" "Quadrant3" (at 144.78 71.6784 0)
+      (effects (font (size 1.27 1.27)) (justify left bottom))
+    )
+    (property "Sheetfile" "quadrant.kicad_sch" (at 144.78 83.1346 0)
+      (effects (font (size 1.27 1.27)) (justify left top))
+    )
+    (pin "DIN" input (at 144.78 77.47 180)
+      (effects (font (size 1.27 1.27)) (justify left))
+    )
+    (pin "DOUT" output (at 166.37 77.47 0)
+      (effects (font (size 1.27 1.27)) (justify right))
+    )
+    (instances
+      (project "analog-clock-module"
+        (path "/894f620e-3404-4a40-a2a7-513bc1d5f99b" (page "40"))
+      )
+    )
+  )
+  (sheet (at 144.78 91.44) (size 21.59 10.16) (fields_autoplaced)
+    (stroke (width 0.1524) (type solid))
+    (fill (color 0 0 0 0.0000))
+    (property "Sheetname" "Quadrant4" (at 144.78 90.7284 0)
+      (effects (font (size 1.27 1.27)) (justify left bottom))
+    )
+    (property "Sheetfile" "quadrant.kicad_sch" (at 144.78 102.1846 0)
+      (effects (font (size 1.27 1.27)) (justify left top))
+    )
+    (pin "DIN" input (at 144.78 96.52 180)
+      (effects (font (size 1.27 1.27)) (justify left))
+    )
+    (pin "DOUT" output (at 166.37 96.52 0)
+      (effects (font (size 1.27 1.27)) (justify right))
+    )
+    (instances
+      (project "analog-clock-module"
+        (path "/894f620e-3404-4a40-a2a7-513bc1d5f99b" (page "59"))
+      )
+    )
+  )
+  (sheet (at 144.78 53.34) (size 21.59 10.16) (fields_autoplaced)
+    (stroke (width 0.1524) (type solid))
+    (fill (color 0 0 0 0.0000))
+    (property "Sheetname" "Quadrant2" (at 144.78 52.6284 0)
+      (effects (font (size 1.27 1.27)) (justify left bottom))
+    )
+    (property "Sheetfile" "quadrant.kicad_sch" (at 144.78 64.0846 0)
+      (effects (font (size 1.27 1.27)) (justify left top))
+    )
+    (pin "DIN" input (at 144.78 58.42 180)
+      (effects (font (size 1.27 1.27)) (justify left))
+    )
+    (pin "DOUT" output (at 166.37 58.42 0)
+      (effects (font (size 1.27 1.27)) (justify right))
+    )
+    (instances
+      (project "analog-clock-module"
+        (path "/894f620e-3404-4a40-a2a7-513bc1d5f99b" (page "21"))
+      )
+    )

Commit message: Took notes after meeting with nick
Parts:
- added ESP101: ~, KenwoodFox:ESP32S_HiLetgo, symbol KenwoodFox:ESP32S_HiLetgo
- added H101, H102, H103, H104: MountingHole_Pad, MountingHole:MountingHole_3.2mm_M3_DIN965_Pad, symbol Mechanical:MountingHole_Pad
Connections:
- new net GND: H101.1, H102.1, H103.1, H104.1

Commit message: bump to k8, inital BOM for nick
Parts:
- added J1: Barrel_Jack_MountingPin, Connector_BarrelJack:BarrelJack_Kycon_KLDX-0202-xC_Horizontal, symbol Connector:Barrel_Jack_MountingPin
- ESP101: LCSC# (none) -> C571181

Commit message: Clean and move
Parts:
- removed J1: Barrel_Jack_MountingPin, Connector_BarrelJack:BarrelJack_Kycon_KLDX-0202-xC_Horizontal, symbol Connector:Barrel_Jack_MountingPin
- added Q101, Q102: 2N7000, Package_TO_SOT_SMD:SOT-23, symbol Transistor_FET:2N7000
- added R101, R102, R103, R104: 10k, Resistor_THT:R_Axial_DIN0309_L9.0mm_D3.2mm_P12.70mm_Horizontal, symbol Device:R_Small
- added U101: ~, Package_SO:SOIC-28W_7.5x17.9mm_P1.27mm, symbol KenwoodFox:HT16K33
- ESP101: LCSC# C571181 -> (none)
Connections:
- net GND: now also ESP101.14 (GND), ESP101.32 (GND), ESP101.38 (GND), U101.28 (VDD)
- net Quadrant1/DIN: now also Q101.3 (D), R102.2
- net +3.3V: now reaches ESP101.1 (3.3V)
- net +3.3V: now also Q101.2 (G), Q102.2 (G), R101.1, R103.1
- net +5V: now reaches ESP101.19 (VIN)
- net +5V: now also R102.1, R104.1
- net LEFT_QUADRANT: now reaches ESP101.27 (RX2/GPIO16)
- net LEFT_QUADRANT: now also Q102.1 (S), R103.2
- net RIGHT_QUADRANT: now reaches ESP101.28 (TX2/GPIO17)
- net RIGHT_QUADRANT: now also Q101.1 (S), R101.2
- net SDA: now reaches ESP101.33 (I2C_SDA/GPIO21)
- net SDA: now also U101.27 (SDA)
- net SCL: now reaches ESP101.36 (I2C_SCL/GPIO22)
- net SCL: now also U101.26 (SCL)
- new net Quadrant3/DIN: Q102.3 (D), R104.2
- no-connect marks 0 -> 2
Other:
- moved on the sheet: ESP101

Commit message: Properly bump to k8
Parts:
- removed U101: ~, Package_SO:SOIC-28W_7.5x17.9mm_P1.27mm, symbol KenwoodFox:HT16K33
Other:
- added sheet Alphanumeric Display (alphadisplay.kicad_sch)
