File: Hardware/analog-clock-module/analog-clock-module.kicad_sch (KiCad schematic)
At the start: 11 parts, among them Q101 2N7000, Q102 2N7000

Commit message: Bump after nick meeting
Parts:
- added J101: PWR, Connector_Wire:SolderWire-0.25sqmm_1x02_P4.2mm_D0.65mm_OD1.7mm_Relief, symbol Connector:Conn_01x02_Pin
Connections:
- net +5V: now also J101.1 (Pin_1)
- net GND: now also J101.2 (Pin_2)
- no-connect marks 2 -> 31

Commit message: Bump
Parts:
- added R1, R2: 500R, Resistor_THT:R_Axial_DIN0309_L9.0mm_D3.2mm_P12.70mm_Horizontal, symbol Device:R_Small
Connections:
- net LEFT_QUADRANT: now also R2.1; no longer Q102.1 (S), R103.2
- net RIGHT_QUADRANT: now also R1.1; no longer Q101.1 (S), R101.2
- new net: Q101.1 (S), R1.2, R101.2
- new net: Q102.1 (S), R103.2, R2.2
Changed lines of the file:
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@@
 	(wire
 		(pts
-			(xy 201.93 78.74) (xy 220.98 78.74)
+			(xy 185.42 78.74) (xy 208.28 78.74)
 		)
 		(stroke
@@
 	(wire
 		(pts
+			(xy 213.36 40.64) (xy 220.98 40.64)
+		)
+		(stroke
+			(width 0)
+			(type default)
+		)
+	)
+	(wire
+		(pts
 			(xy 248.92 59.69) (xy 252.73 59.69)
 		)
@@
 	(wire
 		(pts
+			(xy 213.36 78.74) (xy 220.98 78.74)
+		)
+		(stroke
+			(width 0)
+			(type default)
+		)
+	)
+	(wire
+		(pts
 			(xy 106.68 27.94) (xy 106.68 29.21)
 		)
@@
 	(wire
 		(pts
-			(xy 201.93 40.64) (xy 220.98 40.64)
+			(xy 185.42 40.64) (xy 208.28 40.64)
 		)
 		(stroke
@@
 	)
 	(label "RIGHT_QUADRANT"
-		(at 201.93 40.64 0)
+		(at 185.42 40.64 0)
 		(fields_autoplaced yes)
 		(effects
@@
 	)
 	(label "LEFT_QUADRANT"
-		(at 201.93 78.74 0)
+		(at 185.42 78.74 0)
 		(fields_autoplaced yes)
 		(effects
@@
 	)
 	(symbol
+		(lib_id "Device:R_Small")
+		(at 210.82 40.64 90)
+		(unit 1)
+		(exclude_from_sim no)
+		(in_bom yes)
+		(on_board yes)
+		(dnp no)
+		(fields_autoplaced yes)
+		(property "Reference" "R1"
+			(at 210.82 35.56 90)
+			(effects
+				(font
+					(size 1.27 1.27)
+				)
+			)
+		)
+		(property "Value" "500R"
+			(at 210.82 38.1 90)
+			(effects
+				(font
+					(size 1.27 1.27)
+				)
+			)
+		)
+		(property "Footprint" "Resistor_THT:R_Axial_DIN0309_L9.0mm_D3.2mm_P12.70mm_Horizontal"
+			(at 210.82 40.64 0)
+			(effects
+				(font
+					(size 1.27 1.27)
+				)
+				(hide yes)
+			)
+		)
+		(property "Datasheet" "~"
+			(at 210.82 40.64 0)
+			(effects
+				(font
+					(size 1.27 1.27)
+				)
+				(hide yes)
+			)
+		)
+		(property "Description" ""
+			(at 210.82 40.64 0)
+			(effects
+				(font
+					(size 1.27 1.27)
+				)
+				(hide yes)
+			)
+		)
+		(pin "2"
+		)
+		(pin "1"
+		)
+		(instances
+			(project "analog-clock-module"
+				(path "/894f620e-3404-4a40-a2a7-513bc1d5f99b"
+					(reference "R1")
+					(unit 1)
+				)
+			)
+		)
+	)
+	(symbol
 		(lib_id "power:+5V")
 		(at 241.3 25.4 0)
@@
 					(unit 1)
 				)
+			)
+		)
+	)
+	(symbol
+		(lib_id "Device:R_Small")
+		(at 210.82 78.74 90)
+		(unit 1)
+		(exclude_from_sim no)
+		(in_bom yes)
+		(on_board yes)
+		(dnp no)
+		(fields_autoplaced yes)
+		(property "Reference" "R2"
+			(at 210.82 73.66 90)
+			(effects
+				(font
+					(size 1.27 1.27)
+				)
+			)
+		)
+		(property "Value" "500R"
+			(at 210.82 76.2 90)
+			(effects
+				(font
+					(size 1.27 1.27)
+				)
+			)
+		)
+		(property "Footprint" "Resistor_THT:R_Axial_DIN0309_L9.0mm_D3.2mm_P12.70mm_Horizontal"
+			(at 210.82 78.74 0)
+			(effects
+				(font
+					(size 1.27 1.27)
+				)
+				(hide yes)
+			)
+		)
+		(property "Datasheet" "~"
+			(at 210.82 78.74 0)
+			(effects
+				(font
+					(size 1.27 1.27)
+				)
+				(hide yes)
+			)
+		)
+		(property "Description" ""
+			(at 210.82 78.74 0)
+			(effects
+				(font
+					(size 1.27 1.27)
+				)
+				(hide yes)
+			)
+		)
+		(pin "2"
+		)
+		(pin "1"
+		)
+		(instances
+			(project "analog-clock-module"
+				(path "/894f620e-3404-4a40-a2a7-513bc1d5f99b"
+					(reference "R2")
+					(unit 1)
+				)
