File: Hardware/analog-clock-module/quadrant.kicad_sch (KiCad schematic)
At the start: 0 parts

Commit message: Clean and move
Other:
- removed sheet Hour1
- removed sheet Hour2
- removed sheet Hour3

Commit message: Properly bump to k8
Other:
- added sheet Hour1 (hour.kicad_sch)
- added sheet Hour2 (hour.kicad_sch)
- added sheet Hour3 (hour.kicad_sch)
