File: Hardware/analog-clock-module/ClockInnerHand.kicad_sch (KiCad schematic)
At the start: 10 parts

Commit message: bump
Connections:
- net DOUT: now also D210.1 (DOUT)
Changed lines of the file:
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@@
     (effects (font (size 1.27 1.27)) (justify left bottom))
   )
-  (hierarchical_label "DOUT" (shape output) (at 250.19 93.98 0) (fields_autoplaced)
+  (hierarchical_label "DOUT" (shape output) (at 248.92 93.98 0) (fields_autoplaced)
     (effects (font (size 1.27 1.27)) (justify left))
   )

Commit message: full quadrant
Parts:
- renumbered D201 to D301, D202 to D302, D203 to D303, D204 to D304, D205 to D305, D206 to D306, D207 to D307, D208 to D308, D209 to D309, D210 to D310

Commit message: All done
Parts:
- renumbered D301 to D6101, D302 to D6102, D303 to D6103, D304 to D6104, D305 to D6105, D306 to D6106, D307 to D6107, D308 to D6108, D309 to D6109, D310 to D6110

Commit message: Took notes after meeting with nick
Parts:
- D6101, D6102, D6103, D6104, D6105, D6106, D6107, D6108, D6109, D6110: LCSC# (none) -> C4154875
Changed lines of the file:
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@@
       (effects (font (size 1.27 1.27)) (justify left top) hide)
     )
+    (property "LCSC#" "C4154875" (at 40.64 93.98 0)
+      (effects (font (size 1.27 1.27)) hide)
+    )
     (pin "3")
     (pin "2")
@@
       (effects (font (size 1.27 1.27)) (justify left top) hide)
     )
+    (property "LCSC#" "C4154875" (at 83.82 93.98 0)
+      (effects (font (size 1.27 1.27)) hide)
+    )
     (pin "3")
     (pin "2")
@@
       (effects (font (size 1.27 1.27)) (justify left top) hide)
     )
+    (property "LCSC#" "C4154875" (at 105.41 93.98 0)
+      (effects (font (size 1.27 1.27)) hide)
+    )
     (pin "3")
     (pin "2")
@@
       (effects (font (size 1.27 1.27)) (justify left top) hide)
     )
+    (property "LCSC#" "C4154875" (at 62.23 93.98 0)
+      (effects (font (size 1.27 1.27)) hide)
+    )
     (pin "3")
     (pin "2")
@@
       (effects (font (size 1.27 1.27)) (justify left top) hide)
     )
+    (property "LCSC#" "C4154875" (at 234.95 93.98 0)
+      (effects (font (size 1.27 1.27)) hide)
+    )
     (pin "3")
     (pin "2")
@@
       (effects (font (size 1.27 1.27)) (justify left top) hide)
     )
+    (property "LCSC#" "C4154875" (at 127 93.98 0)
+      (effects (font (size 1.27 1.27)) hide)
+    )
     (pin "3")
     (pin "2")
@@
       (effects (font (size 1.27 1.27)) (justify left top) hide)
     )
+    (property "LCSC#" "C4154875" (at 213.36 93.98 0)
+      (effects (font (size 1.27 1.27)) hide)
+    )
     (pin "3")
     (pin "2")
@@
       (effects (font (size 1.27 1.27)) (justify left top) hide)
     )
+    (property "LCSC#" "C4154875" (at 170.18 93.98 0)
+      (effects (font (size 1.27 1.27)) hide)
+    )
     (pin "3")
     (pin "2")
@@
       (effects (font (size 1.27 1.27)) (justify left top) hide)
     )
+    (property "LCSC#" "C4154875" (at 191.77 93.98 0)
+      (effects (font (size 1.27 1.27)) hide)
+    )
     (pin "3")
     (pin "2")
@@
       (effects (font (size 1.27 1.27)) (justify left top) hide)
     )
+    (property "LCSC#" "C4154875" (at 148.59 93.98 0)
+      (effects (font (size 1.27 1.27)) hide)
+    )
     (pin "3")

Commit message: Clean and move
Parts:
- renumbered D6101 to D2301, D6102 to D2302, D6103 to D2303, D6104 to D2304, D6105 to D2305, D6106 to D2306, D6107 to D2307, D6108 to D2308, D6109 to D2309, D6110 to D2310

Commit message: Properly bump to k8
Parts:
- renumbered D2301 to D6101, D2302 to D6102, D2303 to D6103, D2304 to D6104, D2305 to D6105, D2306 to D6106, D2307 to D6107, D2308 to D6108, D2309 to D6109, D2310 to D6110

Commit message: Bump after nick meeting
Parts:
- renumbered D6101 to D2301, D6102 to D2302, D6103 to D2303, D6104 to D2304, D6105 to D2305, D6106 to D2306, D6107 to D2307, D6108 to D2308, D6109 to D2309, D6110 to D2310
Changed lines of the file:
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@@
 		(on_board yes)
 		(dnp no)
-		(property "Reference" "D6101"
+		(property "Reference" "D2301"
 			(at 48.26 101.6 0)
 			(effects
@@
 		(dnp no)
 		(fields_autoplaced yes)
-		(property "Reference" "#PWR06114"
+		(property "Reference" "#PWR02314"
 			(at 170.18 111.76 0)
 			(effects
@@
 		(on_board yes)
 		(dnp no)
-		(property "Reference" "D6103"
+		(property "Reference" "D2303"
 			(at 91.44 101.6 0)
 			(effects
@@
 		(dnp no)
 		(fields_autoplaced yes)
-		(property "Reference" "#PWR06109"
+		(property "Reference" "#PWR02309"
 			(at 127 86.36 0)
 			(effects
@@
 		(on_board yes)
 		(dnp no)
-		(property "Reference" "D6104"
+		(property "Reference" "D2304"
 			(at 113.03 101.6 0)
 			(effects
@@
 		(dnp no)
 		(fields_autoplaced yes)
-		(property "Reference" "#PWR06119"
+		(property "Reference" "#PWR02319"
 			(at 234.95 86.36 0)
 			(effects
@@
 		(on_board yes)
 		(dnp no)
-		(property "Reference" "D6102"
+		(property "Reference" "D2302"
 			(at 69.85 101.6 0)
 			(effects
@@
 		(on_board yes)
 		(dnp no)
-		(property "Reference" "D6110"
+		(property "Reference" "D2310"
 			(at 242.57 101.6 0)
 			(effects
@@
 		(dnp no)
 		(fields_autoplaced yes)
-		(property "Reference" "#PWR06108"
+		(property "Reference" "#PWR02308"
 			(at 105.41 111.76 0)
 			(effects
@@
 		(dnp no)
 		(fields_autoplaced yes)
-		(property "Reference" "#PWR06115"
+		(property "Reference" "#PWR02315"
 			(at 191.77 86.36 0)
 			(effects
@@
 		(on_board yes)
 		(dnp no)
-		(property "Reference" "D6105"
+		(property "Reference" "D2305"
 			(at 134.62 101.6 0)
 			(effects
@@
 		(dnp no)
 		(fields_autoplaced yes)
-		(property "Reference" "#PWR06116"
+		(property "Reference" "#PWR02316"
 			(at 191.77 111.76 0)
 			(effects
@@
 		(dnp no)
 		(fields_autoplaced yes)
-		(property "Reference" "#PWR06105"
+		(property "Reference" "#PWR02305"
 			(at 83.82 86.36 0)
 			(effects
@@
 		(on_board yes)
 		(dnp no)
-		(property "Reference" "D6109"
+		(property "Reference" "D2309"
 			(at 220.98 101.6 0)
 			(effects
@@
 		(dnp no)
 		(fields_autoplaced yes)
-		(property "Reference" "#PWR06107"
+		(property "Reference" "#PWR02307"
 			(at 105.41 86.36 0)
 			(effects
@@
 		(on_board yes)
 		(dnp no)
-		(property "Reference" "D6107"
+		(property "Reference" "D2307"
 			(at 177.8 101.6 0)
 			(effects
@@
 		(dnp no)
 		(fields_autoplaced yes)
-		(property "Reference" "#PWR06110"
+		(property "Reference" "#PWR02310"
 			(at 127 111.76 0)
 			(effects
@@
 		(dnp no)
 		(fields_autoplaced yes)
-		(property "Reference" "#PWR06101"
+		(property "Reference" "#PWR02301"
 			(at 40.64 86.36 0)
 			(effects
@@
 		(dnp no)
 		(fields_autoplaced yes)
-		(property "Reference" "#PWR06102"
+		(property "Reference" "#PWR02302"
 			(at 40.64 111.76 0)
 			(effects
@@
 		(dnp no)
 		(fields_autoplaced yes)
-		(property "Reference" "#PWR06103"
+		(property "Reference" "#PWR02303"
 			(at 62.23 86.36 0)
 			(effects
@@
 		(dnp no)
 		(fields_autoplaced yes)
-		(property "Reference" "#PWR06117"
+		(property "Reference" "#PWR02317"
 			(at 213.36 86.36 0)
 			(effects
@@
 		(dnp no)
 		(fields_autoplaced yes)
-		(property "Reference" "#PWR06113"
+		(property "Reference" "#PWR02313"
 			(at 170.18 86.36 0)
 			(effects
@@
 		(dnp no)
 		(fields_autoplaced yes)
-		(property "Reference" "#PWR06112"
+		(property "Reference" "#PWR02312"
 			(at 148.59 111.76 0)
 			(effects
@@
 		(dnp no)
 		(fields_autoplaced yes)
-		(property "Reference" "#PWR06104"
+		(property "Reference" "#PWR02304"
 			(at 62.23 111.76 0)
 			(effects
@@
 		(dnp no)
 		(fields_autoplaced yes)
-		(property "Reference" "#PWR06111"
+		(property "Reference" "#PWR02311"
 			(at 148.59 86.36 0)
 			(effects
@@
 		(dnp no)
 		(fields_autoplaced yes)
-		(property "Reference" "#PWR06118"
+		(property "Reference" "#PWR02318"
 			(at 213.36 111.76 0)
 			(effects
@@
 		(on_board yes)
 		(dnp no)
-		(property "Reference" "D6108"
+		(property "Reference" "D2308"
 			(at 199.39 101.6 0)
 			(effects
@@
 		(dnp no)
 		(fields_autoplaced yes)
-		(property "Reference" "#PWR06106"
+		(property "Reference" "#PWR02306"
 			(at 83.82 111.76 0)
 			(effects
@@
 		(on_board yes)
 		(dnp no)
-		(property "Reference" "D6106"
+		(property "Reference" "D2306"
 			(at 156.21 101.6 0)
 			(effects
@@
 		(dnp no)
 		(fields_autoplaced yes)
-		(property "Reference" "#PWR06120"
+		(property "Reference" "#PWR02320"
 			(at 234.95 111.76 0)
 			(effects
